File: VESCmodul/VESC_modul/VESC_modul.kicad_pcb (KiCad board)
At the start: 4 copper layers, 30 x 18 mm, 48 parts, among them U1 DRV8320RS, U2 STM32F405RGTx, U3 PINx6, U4 PINx4, U5 PINx2, U6 PINx6, U7 PINx6, U8 PINx4, U9 PINx6, Y1 ABM3B-8.000-U-T

Commit message: initial commit
Parts:
- removed the C12 at (124.1, 112.0)
- removed the C15 at (109.2, 100.8)
- removed the C19 at (102.0, 108.0)
- removed the C22 at (115.9, 116.6)
- removed the C4 at (127.1, 109.2)
- removed the C7 at (118.5, 112.0)
- removed the R6 at (101.0, 116.6)
- removed the U4 at (119.1, 100.0)
- added C13: 2.2uF 60V, Capacitors_SMD:C_1206, F.Cu at (124.9, 111.7)
- added C16: 15pF, Capacitors_SMD:C_0603, F.Cu at (109.0, 100.8)
- added C21: 2.2uF, Capacitors_SMD:C_0603, F.Cu at (115.4, 105.3)
- added C26: 2.2uF, Capacitors_SMD:C_0603, F.Cu at (102.0, 111.2)
- added C3: 100nF 60V, Capacitors_SMD:C_0603, F.Cu at (126.7, 107.8)
- added C5: 47nF 60V, Capacitors_SMD:C_0603, F.Cu at (126.7, 110.1)
- added C8: 100nF, Capacitors_SMD:C_0603, F.Cu at (116.8, 112.9)
- added R3: 5.6k, Resistors_SMD:R_0603, F.Cu at (101.5, 104.6)
- added R4: 5.6k, Resistors_SMD:R_0603, F.Cu at (101.5, 102.1)
- added R5: 5.6k, Resistors_SMD:R_0603, F.Cu at (101.5, 100.8)
- added R9: 220R, Resistors_SMD:R_0603, F.Cu at (101.0, 116.6)
- added U2: PINx4, user_defined:PINx4-1.27mm, F.Cu at (118.4, 100.0)
- added U7: PINx9, user_defined:PINx9-1.27mm, F.Cu at (112.6, 118.0)
- C1: value GRM32ER71J106KA12L -> 4.7uF
- C2: value 100nF -> 4.7uF; footprint Capacitors_SMD:C_0603 -> Capacitors_SMD:C_1210
- C24: value 100nF -> 2.2uF
- C25: value 2.2uF -> 100nF
- C4: renamed from C3; value 1uF -> 1uF 16V
- R2: value ACAS 5k -> 5.6k; footprint Resistors_SMD:R_Array_Convex_4x0603 -> Resistors_SMD:R_0603
- U9: value PINx6 -> MCP1700-3.3V; footprint user_defined:PINx6-1.27mm -> TO_SOT_Packages_SMD:SOT-23
- moved C23 16.8 mm to (115.9, 116.6), turned to 180 degrees
- moved C20 13.5 mm to (102.0, 108.6), turned to 0 degrees
- moved U9 6.78 mm to (119.0, 115.7), turned to 0 degrees
- moved C25 5.38 mm to (104.1, 104.6), turned to 0 degrees
- moved C2 3.63 mm to (127.3, 102.7), turned to 0 degrees
- moved R6 2.20 mm to (126.4, 113.3)
- moved C24 2.09 mm to (102.0, 106.0)
- moved U3 1.82 mm to (130.0, 105.1)
- moved C1 1.80 mm to (127.4, 105.8)
- moved L1 1.65 mm to (123.4, 115.7)
- moved C12 1.59 mm to (121.5, 115.7)
- moved R2 1.30 mm to (101.5, 103.4), turned to 180 degrees
- moved R7 1.23 mm to (124.1, 113.3), turned to 0 degrees
- moved C4 1.20 mm to (126.7, 108.9)
- moved C19 0.99 mm to (116.7, 105.3), turned to 90 degrees
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- renumbered C9 to C10, C10 to C11, C11 to C12, C13 to C14, C14 to C15, C16 to C19, C21 to C22, C5 to C6, C6 to C7, C8 to C9, R7 to R10, R8 to R11, R9 to R12, R3 to R6, R4 to R7, R5 to R8, U3 to U1, U2 to U10, U5 to U3, U6 to U4, U7 to U5, U8 to U6, U1 to U8
Connections:
- C12 pad 1: VCC -> 5V
- C23 pad 1: AGND_EXT -> GND_EXT
- C23 pad 2: VAA -> VCC
- C25 pad 1: TEMP_MOTOR_EXT -> AGND_EXT
- C25 pad 2: AGND_EXT -> VAA
- L1 pad 1: VCC -> 5V
- R2 pad 1: AGND_EXT -> AN_IN
- R7 pad 1: VCC -> 5V
- U10 pad 11: TEMP_FET_EXT -> AN_IN
- U10 pad 17: AN_IN -> TEMP_FET_EXT
- U9 pad 1: CAN_RX_EXT -> GND_EXT
- U9 pad 2: CAN_TX_EXT -> VCC
- U9 pad 3: USB_DM_EXT -> 5V
Routing:
- net GND_EXT: track 68.7 -> 54.0 mm, vias 24 -> 21
- net 5V: track 0.00 -> 11.1 mm, vias 0 -> 2
- net VDD: track 44.8 -> 37.7 mm
- net AGND_EXT: track 61.9 -> 55.2 mm
- net Net-(C6-Pad1): track 5.28 -> 0.00 mm
- net VCC: track 71.6 -> 76.7 mm
- net AN_IN: track 7.06 -> 10.2 mm
- net TEMP_FET_EXT: track 24.7 -> 22.6 mm, vias 2 -> 1
- net Net-(C19-Pad1): track 5.72 -> 7.68 mm
- net TEMP_MOTOR_EXT: track 11.3 -> 12.6 mm
- net LED_R: track 8.58 -> 7.40 mm
- net VAA: track 34.4 -> 33.3 mm
- net TX_SCL_MOSI_EXT: track 9.86 -> 10.9 mm
- net SH3_EXT: track 22.0 -> 21.1 mm
- net VOLTAGE_3: track 4.93 -> 5.74 mm
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- added copper zone on F.Cu, net 5V
- added copper zone on F.Cu, net Net-(C6-Pad1)
- added copper zone on F.Cu, net VAA
Other:
- board text added: "*LN - Low Noise"
- board text added: "3.3V 3.3V (LN) GND (LN) Curr A Curr B Curr C"
- board text added: "CAN RX CAN TX USB D- USB D+ SWDIO SWCLK 0.1A 3.3V 0.5A 5V GND"
- board text added: "NSS MOSI MISO"
- board text added: "SCK SDA SCL"
- board text added: "SERVO ADC1 RX TX ADC2 ADC3"
- board text added: "SH 1 SH 2 SH 3 TEMP_F GL 3 GH 3 GL 2 GH 2 GL 1 GH 1"
- board text added: "TEMP_M HALL 1 HALL 2 HALL 3"
- board text added: "VESC-Modul"
- board text added: "use for analog readings"
- board text added: "v0.1.2019.02.24"
