File: VESC_modul.sch (KiCad schematic (older format))
At the start: 53 parts, among them U1 PINx6, U10 STM32F405RGTx, U2 PINx4, U3 PINx2, U4 PINx6, U5 PINx6, U6 PINx4, U7 PINx9, U8 DRV8320RS, U9 MCP1700-3.3V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

Commit message: improved GND
Parts:
- removed U5: PINx6, user_defined:PINx6-1.27mm, symbol VESC_modul_lib:PINx6
- added U5: PINx8, user_defined:PINx8-1.27mm, symbol VESC_modul_lib:PINx8
Connections:
- net labels added: GNDD
- wire segments 306 -> 308
Changed lines of the file:
@@
 Sheet 1 1
 Title "VESC Modul"
-Date "2019-03-02"
+Date "2019-03-13"
 Rev "0.1"
 Comp "Fabian Viermetz"
@@
 Wire Wire Line
 	4900 1450 5000 1450
-$Comp
-L power:GND #PWR01
-U 1 1 5C7C49DB
-P 1250 1450
-F 0 "#PWR01" H 1250 1200 50  0001 C CNN
-F 1 "GND" V 1255 1322 50  0000 R CNN
-F 2 "" H 1250 1450 50  0001 C CNN
-F 3 "" H 1250 1450 50  0001 C CNN
-	1    1250 1450
-	0    1    1    0
-$EndComp
 Wire Wire Line
 	2900 1450 1950 1450
@@
 Wire Wire Line
 	4900 1250 5000 1250
-$Comp
-L power:GND #PWR08
-U 1 1 5C994289
-P 3550 3650
-F 0 "#PWR08" H 3550 3400 50  0001 C CNN
-F 1 "GND" H 3555 3477 50  0000 C CNN
-F 2 "" H 3550 3650 50  0001 C CNN
-F 3 "" H 3550 3650 50  0001 C CNN
-	1    3550 3650
-	1    0    0    -1
-$EndComp
 Wire Wire Line
 	3550 3650 3550 3550
@@
 Text GLabel 2800 3350 0    50   Output ~ 0
 FAULT
-$Comp
-L power:GND #PWR06
-U 1 1 5C9BBEBA
-P 2800 3250
-F 0 "#PWR06" H 2800 3000 50  0001 C CNN
-F 1 "GND" V 2805 3122 50  0000 R CNN
-F 2 "" H 2800 3250 50  0001 C CNN
-F 3 "" H 2800 3250 50  0001 C CNN
-	1    2800 3250
-	0    1    1    0
-$EndComp
 Wire Wire Line
 	2800 3250 2900 3250
@@
 Wire Wire Line
 	2800 3050 2900 3050
-$Comp
-L power:GND #PWR03
-U 1 1 5CB6ACFF
-P 2800 2350
-F 0 "#PWR03" H 2800 2100 50  0001 C CNN
-F 1 "GND" V 2805 2222 50  0000 R CNN
-F 2 "" H 2800 2350 50  0001 C CNN
-F 3 "" H 2800 2350 50  0001 C CNN
-	1    2800 2350
-	0    1    1    0
-$EndComp
-$Comp
-L power:GND #PWR04
-U 1 1 5CB6AD48
-P 2800 2450
-F 0 "#PWR04" H 2800 2200 50  0001 C CNN
-F 1 "GND" V 2805 2322 50  0000 R CNN
-F 2 "" H 2800 2450 50  0001 C CNN
-F 3 "" H 2800 2450 50  0001 C CNN
-	1    2800 2450
-	0    1    1    0
-$EndComp
-$Comp
-L power:GND #PWR05
-U 1 1 5CB6ADF9
-P 2800 3150
-F 0 "#PWR05" H 2800 2900 50  0001 C CNN
-F 1 "GND" V 2805 3022 50  0000 R CNN
-F 2 "" H 2800 3150 50  0001 C CNN
-F 3 "" H 2800 3150 50  0001 C CNN
-	1    2800 3150
-	0    1    1    0
-$EndComp
 Wire Wire Line
 	2800 2350 2900 2350
@@
 Text GLabel 1300 4700 2    50   BiDi ~ 0
 AGND_EXT
-Text GLabel 1300 4000 2    50   BiDi ~ 0
-GND_EXT
 Text GLabel 1300 4600 2    50   Output ~ 0
 I1_EXT
@@
 $EndComp
 $Comp
-L VESC_modul_lib:PINx6 U5
-U 1 1 5C9653B1
-P 1100 5550
-F 0 "U5" H 1131 6025 50  0000 C CNN
-F 1 "PINx6" H 1131 5934 50  0000 C CNN
-F 2 "user_defined:PINx6-1.27mm" H 1100 5550 50  0001 C CNN
-F 3 "" H 1100 5550 50  0001 C CNN
-	1    1100 5550
-	1    0    0    -1
-$EndComp
-$Comp
 L VESC_modul_lib:PINx2 U3
 U 1 1 5C9656AA
@@
 Wire Wire Line
 	1450 1850 1700 1850
+$Comp
+L power:GND #PWR06
+U 1 1 5C9BBEBA
+P 2800 3250
+F 0 "#PWR06" H 2800 3000 50  0001 C CNN
+F 1 "GND" V 2805 3122 50  0000 R CNN
+F 2 "" H 2800 3250 50  0001 C CNN
+F 3 "" H 2800 3250 50  0001 C CNN
+	1    2800 3250
+	0    1    1    0
+$EndComp
+$Comp
+L VESC_modul_lib:PINx8 U5
+U 1 1 5C8BB595
+P 1100 5550
+F 0 "U5" H 1131 6125 50  0000 C CNN
+F 1 "PINx8" H 1131 6034 50  0000 C CNN
+F 2 "user_defined:PINx8-1.27mm" H 1100 5650 50  0001 C CNN
+F 3 "" H 1100 5650 50  0001 C CNN
+	1    1100 5550
+	1    0    0    -1
+$EndComp
+$Comp
+L power:GND #PWR0101
+U 1 1 5C8BB6E2
+P 1300 5900
+F 0 "#PWR0101" H 1300 5650 50  0001 C CNN
+F 1 "GND" V 1305 5772 50  0000 R CNN
+F 2 "" H 1300 5900 50  0001 C CNN
+F 3 "" H 1300 5900 50  0001 C CNN
+	1    1300 5900
+	0    -1   -1   0
+$EndComp
+$Comp
+L power:GNDREF #PWR0102
+U 1 1 5C8BC2F5
+P 1300 5200
+F 0 "#PWR0102" H 1300 4950 50  0001 C CNN
+F 1 "GNDREF" V 1300 4950 50  0000 C CNN
+F 2 "" H 1300 5200 50  0001 C CNN
+F 3 "" H 1300 5200 50  0001 C CNN
+	1    1300 5200
+	0    -1   -1   0
+$EndComp
+Wire Wire Line
+	1200 5200 1300 5200
+Wire Wire Line
+	1200 5900 1300 5900
+$Comp
+L power:GNDD #PWR0103
+U 1 1 5C908858
+P 2800 3150
+F 0 "#PWR0103" H 2800 2900 50  0001 C CNN
+F 1 "GNDD" V 2804 3040 50  0000 R CNN
+F 2 "" H 2800 3150 50  0001 C CNN
+F 3 "" H 2800 3150 50  0001 C CNN
+	1    2800 3150
+	0    1    1    0
+$EndComp
+$Comp
+L power:GNDD #PWR0104
+U 1 1 5C908909
+P 2800 2350
+F 0 "#PWR0104" H 2800 2100 50  0001 C CNN
+F 1 "GNDD" V 2804 2240 50  0000 R CNN
+F 2 "" H 2800 2350 50  0001 C CNN
+F 3 "" H 2800 2350 50  0001 C CNN
+	1    2800 2350
+	0    1    1    0
+$EndComp
+$Comp
+L power:GNDD #PWR0105
+U 1 1 5C90897E
+P 2800 2450
+F 0 "#PWR0105" H 2800 2200 50  0001 C CNN
+F 1 "GNDD" V 2804 2340 50  0000 R CNN
+F 2 "" H 2800 2450 50  0001 C CNN
+F 3 "" H 2800 2450 50  0001 C CNN
+	1    2800 2450
+	0    1    1    0
+$EndComp
+$Comp
+L power:GNDD #PWR0106
+U 1 1 5C9089F3
+P 1250 1450
+F 0 "#PWR0106" H 1250 1200 50  0001 C CNN
+F 1 "GNDD" V 1254 1340 50  0000 R CNN
+F 2 "" H 1250 1450 50  0001 C CNN
+F 3 "" H 1250 1450 50  0001 C CNN
+	1    1250 1450
+	0    1    1    0
+$EndComp
+$Comp
+L power:GNDD #PWR0107
+U 1 1 5C908BA7
+P 3550 3650
+F 0 "#PWR0107" H 3550 3400 50  0001 C CNN
+F 1 "GNDD" H 3554 3495 50  0000 C CNN
+F 2 "" H 3550 3650 50  0001 C CNN
+F 3 "" H 3550 3650 50  0001 C CNN
+	1    3550 3650
+	1    0    0    -1
+$EndComp
+$Comp
+L power:GNDD #PWR0108
+U 1 1 5C90961C
+P 1300 4000
+F 0 "#PWR0108" H 1300 3750 50  0001 C CNN
+F 1 "GNDD" V 1304 3890 50  0000 R CNN
+F 2 "" H 1300 4000 50  0001 C CNN
+F 3 "" H 1300 4000 50  0001 C CNN
+	1    1300 4000
+	0    -1   -1   0
+$EndComp
 $EndSCHEMATC
